File: Rotary Encoder Breakout Board.sch (KiCad schematic (older format))
At the start: 32 parts, among them J1 B5B-XH-A_LF__SN_, Q1 AO3401A, Q2 AO3401A, Q3 AO3401A, SW1 Rotary_Encoder_Switch, U1 SN74HC14DR

Commit message: simplified schematic + updated pcb + added pours, outline and mounting holes
Parts:
- removed Q1, Q2, Q3: AO3401A, digikey-footprints:SOT-23-3, symbol dk_Transistors-FETs-MOSFETs-Single:AO3401A
- removed R5, R7, R9: 510, Resistor_SMD:R_0805_2012Metric, symbol Device:R
- added H1, H2, H3, H4: MountingHole, MountingHole:MountingHole_4.3mm_M4_ISO7380, symbol Mechanical:MountingHole
- R11, R13, R15: value 1k8 -> 1k
- SW1: footprint SnapEDA:XDCR_PEC11R-4215F-S0024 -> Rotary_Encoder:RotaryEncoder_Alps_EC11E-Switch_Vertical_H20mm
Connections:
- net 2Y: now also R11.1
- net 4Y: now also R15.1
- net 5Y: now also R13.1
- net GND: no longer R11.1, R13.1, R15.1
- net VCC: now also D1.2 (A), D2.2 (A), D3.2 (A)
Other:
- moved on the sheet: D1, D2, D3, R11, R13, R15

Commit message: work in progress
Parts:
- J1: footprint digikey-footprints:PinHeader_1x5_P2.5mm_Drill1.1mm -> Connector_PinHeader_2.54mm:PinHeader_1x05_P2.54mm_Vertical
Changed lines of the file:
@@
 F 0 "J1" V 9091 2122 50  0000 R CNN
 F 1 "B5B-XH-A_LF__SN_" V 9000 2122 50  0000 R CNN
-F 2 "digikey-footprints:PinHeader_1x5_P2.5mm_Drill1.1mm" H 9050 2450 60  0001 L CNN
+F 2 "Connector_PinHeader_2.54mm:PinHeader_1x05_P2.54mm_Vertical" H 9050 2450 60  0001 L CNN
 F 3 "http://www.jst-mfg.com/product/pdf/eng/eXH.pdf" H 9050 2550 60  0001 L CNN
 F 4 "455-2270-ND" H 9050 2650 60  0001 L CNN "Digi-Key_PN"

Commit message: changed led footprint + added cast. holes + placed labels + pin header
Parts:
- D1, D2, D3: footprint LED_SMD:LED_0201_0603Metric -> LED_SMD:LED_1206_3216Metric
Changed lines of the file:
@@
 F 0 "D1" V 3339 4082 50  0000 R CNN
 F 1 "LED" V 3248 4082 50  0000 R CNN
-F 2 "LED_SMD:LED_0201_0603Metric" H 3300 4200 50  0001 C CNN
+F 2 "LED_SMD:LED_1206_3216Metric" H 3300 4200 50  0001 C CNN
 F 3 "~" H 3300 4200 50  0001 C CNN
 	1    3300 4200
@@
 F 0 "D2" V 6439 4082 50  0000 R CNN
 F 1 "LED" V 6348 4082 50  0000 R CNN
-F 2 "LED_SMD:LED_0201_0603Metric" H 6400 4200 50  0001 C CNN
+F 2 "LED_SMD:LED_1206_3216Metric" H 6400 4200 50  0001 C CNN
 F 3 "~" H 6400 4200 50  0001 C CNN
 	1    6400 4200
@@
 F 0 "D3" V 9539 4082 50  0000 R CNN
 F 1 "LED" V 9448 4082 50  0000 R CNN
-F 2 "LED_SMD:LED_0201_0603Metric" H 9500 4200 50  0001 C CNN
+F 2 "LED_SMD:LED_1206_3216Metric" H 9500 4200 50  0001 C CNN
 F 3 "~" H 9500 4200 50  0001 C CNN
 	1    9500 4200
